File: projects/proto1/proto1.kicad_pcb (KiCad board)
At the start: 4 copper layers, 170 parts, among them J1 ATRANS, J13 MS_SEL, J14 AUDIO_DATA, J15 STX-4335-5BGP-S1, J2 Bus_ISA_16bit, J3 Bus_ISA_16bit, J6 IDC_FDD, J7 IDC_PATA, J8 KMDGX-6SG_P-S4N, U1 MC68030R, U10 DP8440, U11 74LS245, U12 PAL16L8, U13 PAL16L8, U14 74LS245, U15 74LS245, U16 74LS245, U17 74LS245, U2 MC68882FN, U22 PC8477BV, U23 VT82C42, U29 74LS245, U30 74LS245, U31 74LS573, U32 MC68440FN, U33 74LS245, U34 74LS573, U35 74LS00, U36 74LS139, U37 74LS148, U38 74LS245, U39 74LS245, U40 74LS573, U41 MC68440FN, U42 74LS245, U43 74LS573, U44 74LS148, U46 MC68901P, U47 MC68901P, U49 EPM7128SLC84-15, U5 74LS245, U51 CS4231A, U52 74LS245, U53 74LS245, U54 MC33078, U55 MC33078, U6 SIMM72, U7 SIMM72, U8 74LS245, U9 74LS245, X1 10M, Y2 16.9344M, Y3 24.576M

Commit message: Renamed CMC to SCU, changed verification method to cocotb, and modified pcb schematic
Parts:
- removed C100, C101, C102, C104, C79, C80, C84, C99: 1u, Capacitor_THT:CP_Radial_D5.0mm_P2.50mm
- removed C103, C98: 47p, Capacitor_THT:C_Disc_D4.3mm_W1.9mm_P5.00mm
- removed C105, C69, C70, C77, C78, C81, C82, C83, C85, C87, C95: 100n, Capacitor_THT:C_Disc_D4.3mm_W1.9mm_P5.00mm
- removed C71, C72, C73, C74: 20p, Capacitor_THT:C_Disc_D4.3mm_W1.9mm_P5.00mm
- removed C75, C76: 1n, Capacitor_THT:C_Disc_D4.3mm_W1.9mm_P5.00mm
- removed C86, C88, C91, C93: 10u, Capacitor_THT:CP_Radial_D5.0mm_P2.50mm
- removed C89, C92, C96, C97: 1u, Capacitor_THT:C_Disc_D4.3mm_W1.9mm_P5.00mm
- removed C90, C94: 1.2n, Capacitor_THT:C_Disc_D4.3mm_W1.9mm_P5.00mm
- removed J15: STX-4335-5BGP-S1, STX43355BGPS1:STX43355BGPS1
- removed RN12: 10k, Resistor_THT:R_Array_SIP5
- removed RN14: 33, Package_DIP:DIP-8_W7.62mm
- removed U39, U52, U53: 74LS245, Package_DIP:DIP-20_W7.62mm_Socket
- removed U46, U47: MC68901P, Package_DIP:DIP-48_W15.24mm_Socket
- removed U49: EPM7128SLC84-15, Package_LCC:PLCC-84_THT-Socket
- removed U51: CS4231A, Package_LCC:PLCC-68_THT-Socket
- removed U54, U55: MC33078, Package_DIP:DIP-8_W7.62mm_Socket
- added C17: 1u, Capacitor_THT:C_Disc_D4.3mm_W1.9mm_P5.00mm, F.Cu at (-235.8, 117.0)
- added C18: 1u, Capacitor_THT:C_Disc_D4.3mm_W1.9mm_P5.00mm, F.Cu at (-235.8, 120.5)
- added C30: 1u, Capacitor_THT:CP_Radial_D5.0mm_P2.50mm, F.Cu at (-264.6, 156.9)
- added C31: 1u, Capacitor_THT:CP_Radial_D5.0mm_P2.50mm, F.Cu at (-264.6, 163.4)
- added C32: 100n, Capacitor_THT:C_Disc_D4.3mm_W1.9mm_P5.00mm, F.Cu at (-273.2, 169.1)
- added C33: 100n, Capacitor_THT:C_Disc_D4.3mm_W1.9mm_P5.00mm, F.Cu at (-273.2, 172.6)
- added C34: 100n, Capacitor_THT:C_Disc_D4.3mm_W1.9mm_P5.00mm, F.Cu at (-273.2, 176.0)
- added C35: 1u, Capacitor_THT:CP_Radial_D5.0mm_P2.50mm, F.Cu at (-264.6, 170.0)
- added C36: 20p, Capacitor_THT:C_Disc_D4.3mm_W1.9mm_P5.00mm, F.Cu at (-273.2, 179.5)
- added C37: 20p, Capacitor_THT:C_Disc_D4.3mm_W1.9mm_P5.00mm, F.Cu at (-273.2, 182.9)
- added C38: 100n, Capacitor_THT:C_Disc_D4.3mm_W1.9mm_P5.00mm, F.Cu at (-273.2, 186.4)
- added C42: 1n, Capacitor_THT:C_Disc_D4.3mm_W1.9mm_P5.00mm, F.Cu at (-273.2, 193.3)
- added C43: 1n, Capacitor_THT:C_Disc_D4.3mm_W1.9mm_P5.00mm, F.Cu at (-273.2, 196.7)
- added C44: 1.2n, Capacitor_THT:C_Disc_D4.3mm_W1.9mm_P5.00mm, F.Cu at (-184.7, 174.4)
- added C61: 100n, Capacitor_THT:C_Disc_D4.3mm_W1.9mm_P5.00mm, F.Cu at (-235.8, 206.5)
- added C62: 100n, Capacitor_THT:C_Disc_D4.3mm_W1.9mm_P5.00mm, F.Cu at (-235.8, 209.9)
- added C63: 100n, Capacitor_THT:C_Disc_D4.3mm_W1.9mm_P5.00mm, F.Cu at (-235.8, 213.4)
- added C64: 100n, Capacitor_THT:C_Disc_D4.3mm_W1.9mm_P5.00mm, F.Cu at (-235.8, 216.8)
- added C65: 100n, Capacitor_THT:C_Disc_D4.3mm_W1.9mm_P5.00mm, F.Cu at (-235.8, 220.3)
- added C66: 100n, Capacitor_THT:C_Disc_D4.3mm_W1.9mm_P5.00mm, F.Cu at (-235.8, 223.7)
- added H1: MH, MountingHole:MountingHole_3.2mm_M3_Pad, F.Cu at (-199.5, 208.2)
- added H2: MH, MountingHole:MountingHole_3.2mm_M3_Pad, F.Cu at (-199.5, 216.1)
- added H3: MH, MountingHole:MountingHole_3.2mm_M3_Pad, F.Cu at (-191.6, 208.2)
- added H4: MH, MountingHole:MountingHole_3.2mm_M3_Pad, F.Cu at (-191.6, 216.1)
- added H5: MH, MountingHole:MountingHole_3.2mm_M3_Pad, F.Cu at (-183.6, 208.2)
- added H6: MH, MountingHole:MountingHole_3.2mm_M3_Pad, F.Cu at (-183.6, 216.1)
- added H7: MH, MountingHole:MountingHole_3.2mm_M3_Pad, F.Cu at (-175.7, 208.2)
- added H8: MH, MountingHole:MountingHole_3.2mm_M3_Pad, F.Cu at (-175.7, 216.1)
- added J10: TIMER4-7, Connector_PinHeader_2.54mm:PinHeader_1x05_P2.54mm_Vertical, F.Cu at (-147.8, 208.5)
- added J11: AUDIO_DATA, Connector_PinHeader_2.54mm:PinHeader_2x05_P2.54mm_Vertical, F.Cu at (-257.7, 155.9)
- added J12: STX-4335-5BGP-S1, STX43355BGPS1:STX43355BGPS1, F.Cu at (284.5, 73.7)
- added J4: 5747840-4, 57478404:57478404, F.Cu at (281.9, 163.0)
- added J5: 5747840-4, 57478404:57478404, F.Cu at (281.9, 127.4)
- added J9: TIMER0-3, Connector_PinHeader_2.54mm:PinHeader_1x05_P2.54mm_Vertical, F.Cu at (-152.5, 208.5)
- added L5: L, Inductor_THT:L_Axial_L9.5mm_D4.0mm_P5.08mm_Vertical_Fastron_SMCC, F.Cu at (-179.3, 118.7)
- added R1: 10k, Resistor_THT:R_Axial_DIN0204_L3.6mm_D1.6mm_P7.62mm_Horizontal, F.Cu at (-217.0, 152.8)
- added R2: 55, Resistor_THT:R_Axial_DIN0204_L3.6mm_D1.6mm_P7.62mm_Horizontal, F.Cu at (-217.0, 155.9)
- added R3: 330, Resistor_THT:R_Axial_DIN0204_L3.6mm_D1.6mm_P7.62mm_Horizontal, F.Cu at (-217.0, 159.1)
- added R4: 330, Resistor_THT:R_Axial_DIN0204_L3.6mm_D1.6mm_P7.62mm_Horizontal, F.Cu at (-217.0, 162.2)
- added U19: MC146818P, Package_DIP:DIP-24_W10.16mm, F.Cu at (167.0, 142.2)
- added U20: 74LS348, Package_DIP:DIP-16_W7.62mm_Socket, F.Cu at (-164.5, 208.3)
- added U21: MC68901P, Package_DIP:DIP-48_W15.24mm_Socket, F.Cu at (203.2, 170.2)
- added U24: PAL16L8, Package_DIP:DIP-20_W7.62mm_Socket, F.Cu at (-152.7, 174.8)
- added U26: CS4231A, Package_LCC:PLCC-68_THT-Socket, F.Cu at (231.1, 27.9)
- added U27: MC33078, Package_DIP:DIP-8_W7.62mm_Socket, F.Cu at (-184.2, 192.1)
- added U28: MC33078, Package_DIP:DIP-8_W7.62mm_Socket, F.Cu at (-162.8, 114.0)
- added U3: SIMM72, m68k-hbc-conn:SIMM72, F.Cu at (228.6, 182.9)
- added U4: SIMM72, m68k-hbc-conn:SIMM72, F.Cu at (228.6, 193.0)
- added U45: 74LS573, Package_DIP:DIP-20_W7.62mm_Socket, F.Cu at (104.1, 190.5)
- added X2: 4M, Oscillator:Oscillator_DIP-14, F.Cu at (177.8, 157.5)
- added X3: 3.6864M, Oscillator:Oscillator_DIP-14, F.Cu at (233.7, 74.9)
- added X4: 8M, Oscillator:Oscillator_DIP-14, F.Cu at (208.3, 74.9)
- added Y1: 14.31818M, Crystal:Crystal_HC49-4H_Vertical, F.Cu at (272.0, 251.5)
- C11, C12, C14, C15, C16, C19, C46, C50, C55, C58: value 100n -> 1u
- C24: value 100n -> 47n
- C26, C27: value 100n -> 20p
- C39, C41, C45, C51: value 100n -> 10u; footprint Capacitor_THT:C_Disc_D4.3mm_W1.9mm_P5.00mm -> Capacitor_THT:CP_Radial_D5.0mm_P2.50mm
- C47, C49, C54, C56, C59: value 100n -> 1u; footprint Capacitor_THT:C_Disc_D4.3mm_W1.9mm_P5.00mm -> Capacitor_THT:CP_Radial_D5.0mm_P2.50mm
- C52: value 100n -> 1.2n
- C53, C60: value 100n -> 47p
- J1: value ATRANS -> Bus_ISA_16bit; footprint Connector_PinHeader_2.54mm:PinHeader_2x10_P2.54mm_Vertical -> m68k-hbc-conn:ATA_16bit
- J14: value AUDIO_DATA -> IDC_PATA; footprint Connector_PinHeader_2.54mm:PinHeader_2x05_P2.54mm_Vertical -> Connector_IDC:IDC-Header_2x20_P2.54mm_Vertical
- J7: value IDC_PATA -> KMDGX-6SG_P-S4N; footprint Connector_IDC:IDC-Header_2x20_P2.54mm_Vertical -> KMDGX6SGPS4N:KMDGX6SGPS4N
- J8: value KMDGX-6SG_P-S4N -> ATX-24; footprint KMDGX6SGPS4N:KMDGX6SGPS4N -> Connector_Molex:Molex_Mini-Fit_Jr_5566-24A_2x12_P4.20mm_Vertical
- R10: value 1.5k -> 47k
- R11, R6: value 11k -> 1.5k
- R14: value 22k -> 11k
- R15, R9: value 47k -> 22k
- R18: value 22k -> 47k
- R7: value 1.5k -> 11k
- RN11: footprint Resistor_THT:R_Array_SIP7 -> Resistor_THT:R_Array_SIP5
- RN3: value 10 -> 10k; footprint Package_DIP:DIP-8_W7.62mm -> Resistor_THT:R_Array_SIP10
- RN4: value 10 -> 4.7k; footprint Package_DIP:DIP-8_W7.62mm -> Resistor_THT:R_Array_SIP8
- RN5: value 10k -> 4.7k; footprint Resistor_THT:R_Array_SIP10 -> Resistor_THT:R_Array_SIP7
- RN6: footprint Resistor_THT:R_Array_SIP8 -> Resistor_THT:R_Array_SIP7
- RN7: value 4.7k -> 10k; footprint Resistor_THT:R_Array_SIP7 -> Resistor_THT:R_Array_SIP9
- RN8: value 4.7k -> 33; footprint Resistor_THT:R_Array_SIP7 -> Package_DIP:DIP-8_W7.62mm
- U10: value DP8440 -> 74LS00; footprint Package_LCC:PLCC-84_THT-Socket -> Package_DIP:DIP-14_W7.62mm_Socket
- U11: value 74LS245 -> MC68681P; footprint Package_DIP:DIP-20_W7.62mm_Socket -> Package_DIP:DIP-40_W15.24mm_Socket
- U12: value PAL16L8 -> MAX232; footprint Package_DIP:DIP-20_W7.62mm_Socket -> Package_DIP:DIP-16_W7.62mm_Socket
- U13: value PAL16L8 -> PC8477BV; footprint Package_DIP:DIP-20_W7.62mm_Socket -> Package_LCC:PLCC-68_THT-Socket
- U14: value 74LS245 -> VT82C42; footprint Package_DIP:DIP-20_W7.62mm_Socket -> Package_DIP:DIP-40_W15.24mm_Socket
- U15: value 74LS245 -> MX8315MC; footprint Package_DIP:DIP-20_W7.62mm_Socket -> Package_DIP:DIP-14_W7.62mm_Socket
- U16: value 74LS245 -> SYS_Header; footprint Package_DIP:DIP-20_W7.62mm_Socket -> Connector_PinHeader_2.54mm:PinHeader_2x06_P2.54mm_Vertical
- U17: value 74LS245 -> 74LS04; footprint Package_DIP:DIP-20_W7.62mm_Socket -> Package_DIP:DIP-14_W7.62mm_Socket
- U22: value PC8477BV -> MC68901P; footprint Package_LCC:PLCC-68_THT-Socket -> Package_DIP:DIP-48_W15.24mm_Socket
- U23: value VT82C42 -> PAL16L8; footprint Package_DIP:DIP-40_W15.24mm_Socket -> Package_DIP:DIP-20_W7.62mm_Socket
- U29: value 74LS245 -> EPF6016QC240; footprint Package_DIP:DIP-20_W7.62mm_Socket -> Package_QFP:PQFP-240_32.1x32.1mm_P0.5mm
- U30, U33: value 74LS245 -> 74LS573
- U31: value 74LS573 -> 74LS245
- U32, U41: value MC68440FN -> 74LS245; footprint Package_LCC:PLCC-68_THT-Socket -> Package_DIP:DIP-20_W7.62mm_Socket
- U35: value 74LS00 -> 74LS148; footprint Package_DIP:DIP-14_W7.62mm_Socket -> Package_DIP:DIP-16_W7.62mm_Socket
- U36: value 74LS139 -> MC68440FN; footprint Package_DIP:DIP-16_W7.62mm_Socket -> Package_LCC:PLCC-68_THT-Socket
- U37: value 74LS148 -> MC68440FN; footprint Package_DIP:DIP-16_W7.62mm_Socket -> Package_LCC:PLCC-68_THT-Socket
- U38: value 74LS245 -> 74LS139; footprint Package_DIP:DIP-20_W7.62mm_Socket -> Package_DIP:DIP-16_W7.62mm_Socket
- U40: value 74LS573 -> 74LS04; footprint Package_DIP:DIP-20_W7.62mm_Socket -> Package_DIP:DIP-14_W7.62mm_Socket
- U44: value 74LS148 -> 74LS245; footprint Package_DIP:DIP-16_W7.62mm_Socket -> Package_DIP:DIP-20_W7.62mm_Socket
- U5: value 74LS245 -> SIMM72; footprint Package_DIP:DIP-20_W7.62mm_Socket -> m68k-hbc-conn:SIMM72
- U7: value SIMM72 -> SST39SF040; footprint m68k-hbc-conn:SIMM72 -> Package_DIP:DIP-32_W15.24mm_Socket
- U8: value 74LS245 -> SST39SF040; footprint Package_DIP:DIP-20_W7.62mm_Socket -> Package_DIP:DIP-32_W15.24mm_Socket
- U9: value 74LS245 -> MAX232; footprint Package_DIP:DIP-20_W7.62mm_Socket -> Package_DIP:DIP-16_W7.62mm_Socket
- Y2: value 16.9344M -> 24.576M
- Y3: value 24.576M -> 16.9344M
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Connections:
- C11 pad 1: GND -> Net-(U9-C1+)
- C11 pad 2: +5V -> Net-(U9-C1-)
- C12 pad 1: GND -> Net-(U9-C2+)
- C12 pad 2: +5V -> Net-(U9-C2-)
- C14 pad 1: +5V -> Net-(U9-VS+)
- C15 pad 1: +5V -> Net-(U9-VS-)
- C16 pad 1: GND -> Net-(U12-C1+)
- C16 pad 2: +5V -> Net-(U12-C1-)
- C19 pad 1: GND -> Net-(U12-VS-)
- C19 pad 2: +5V -> GND
- C24 pad 1: GND -> Net-(U15-CAP)
- C24 pad 2: +5V -> GND
- C26 pad 1: GND -> /audio/XTAL1O
- C26 pad 2: +5V -> GND
- C27 pad 1: GND -> /audio/XTAL2O
- C27 pad 2: +5V -> GND
- C39 pad 1: +5V -> /audio/VREFI
- C39 pad 2: GND -> GNDA
- C40 pad 1: +5V -> GNDA
- C40 pad 2: GND -> /audio/VREF
- C41 pad 1: +5V -> /audio/VREF
- C41 pad 2: GND -> GNDA
- C45 pad 1: GND -> Net-(C45-Pad1)
- C45 pad 2: +5V -> GNDA
- C46 pad 1: GND -> /audio/LMIC
- C46 pad 2: +5V -> Net-(C44-Pad2)
- C47 pad 1: GND -> Net-(U27A-+)
- C47 pad 2: +5V -> Net-(J13-Pin_4)
- C48 pad 1: GND -> +5VA
- C48 pad 2: +5V -> GNDA
- C49 pad 1: GND -> Net-(U27B-+)
- C49 pad 2: +5V -> Net-(J13-Pin_3)
- C50 pad 1: GND -> /audio/RMIC
- C50 pad 2: +5V -> Net-(C50-Pad2)
- C51 pad 1: GND -> Net-(C51-Pad1)
- C51 pad 2: +5V -> GNDA
- C52 pad 1: +5V -> Net-(U27B--)
- C52 pad 2: GND -> Net-(C50-Pad2)
- C53 pad 1: GND -> Net-(U28A--)
- C53 pad 2: +5V -> Net-(C53-Pad2)
- C54 pad 1: GND -> Net-(C54-Pad1)
- C54 pad 2: +5V -> Net-(C54-Pad2)
- C55 pad 1: GND -> /audio/LLINE
- C55 pad 2: +5V -> Net-(C53-Pad2)
- C56 pad 1: GND -> Net-(U28A-+)
- C56 pad 2: +5V -> GNDA
- C57 pad 1: GND -> +5VA
- C57 pad 2: +5V -> GNDA
- C58 pad 1: GND -> /audio/RLINE
- C58 pad 2: +5V -> Net-(C58-Pad2)
- C59 pad 1: +5V -> Net-(C59-Pad1)
- C59 pad 2: GND -> Net-(C59-Pad2)
- C60 pad 1: GND -> Net-(U28B--)
- C60 pad 2: +5V -> Net-(C58-Pad2)
- C8 pad 1: +5V -> GND
- C8 pad 2: GND -> +5V
- J1 pad 1: /dram/C8 -> GND
- J1 pad 10: A22 -> GND
- J1 pad 11: /dram/R9 -> /isa/~{SMEMW}
- J1 pad 12: A23 -> /isa/~{SMEMR}
- J1 pad 13: /dram/R10 -> /isa/~{IOW}
- J1 pad 14: A24 -> /isa/~{IOR}
- J1 pad 15: /dram/R11 -> /isa/~{DACK3}
- J1 pad 16: A25 -> /isa/DRQ3
- J1 pad 17: /dram/B1 -> /isa/~{DACK1}
- J1 pad 18: A26 -> /isa/DRQ1
- J1 pad 19: /dram/B0 -> /isa/~{REFRESH}
- J1 pad 2: A10 -> RST
- J1 pad 20: A27 -> 8MHz
- J1 pad 3: /dram/C9 -> +5V
- J1 pad 4: A11 -> IRQ2
- J1 pad 5: /dram/C10 -> unconnected-(J1--5V-Pad5)
- J1 pad 6: A12 -> /isa/DRQ2
- J1 pad 7: /dram/C11 -> -12V
- J1 pad 8: A21 -> /isa/~{NOWS}
- J1 pad 9: /dram/R8 -> +12V
- J14 pad 1: +5V -> ~{RST}
- J14 pad 10: GND -> /isa/BD11
- J14 pad 2: GND -> unconnected-(J14-GND-Pad2)
- J14 pad 3: Net-(J14-Pin_3) -> /isa/BD7
- J14 pad 4: GND -> /isa/BD8
- J14 pad 5: Net-(J14-Pin_5) -> /isa/BD6
- J14 pad 6: GND -> /isa/BD9
- J14 pad 7: Net-(J14-Pin_7) -> /isa/BD5
- J14 pad 8: GND -> /isa/BD10
- J14 pad 9: Net-(J14-Pin_9) -> /isa/BD4
- J2 pad 32: unconnected-(J2-IO-Pad32) -> /isa/~{IOCHCK}
- J2 pad 33: BD23 -> /isa/BD7
- J2 pad 34: BD22 -> /isa/BD6
- J2 pad 35: BD21 -> /isa/BD5
- J2 pad 36: BD20 -> /isa/BD4
- J2 pad 37: BD19 -> /isa/BD3
- J2 pad 38: BD18 -> /isa/BD2
- J2 pad 39: BD17 -> /isa/BD1
- J2 pad 40: BD16 -> /isa/BD0
- J2 pad 43: BA19 -> /isa/BA19
- J2 pad 44: BA18 -> /isa/BA18
- J2 pad 45: BA17 -> /isa/BA17
- J2 pad 46: BA16 -> /isa/BA16
- J2 pad 47: BA15 -> /isa/BA15
- J2 pad 48: BA14 -> /isa/BA14
- J2 pad 49: BA13 -> /isa/BA13
- J2 pad 50: BA12 -> /isa/BA12
- J2 pad 51: BA11 -> /isa/BA11
- J2 pad 52: BA10 -> /isa/BA10
- J2 pad 53: BA9 -> /isa/BA9
- J2 pad 54: BA8 -> /isa/BA8
- J2 pad 55: BA7 -> /isa/BA7
- J2 pad 56: BA6 -> /isa/BA6
- J2 pad 57: BA5 -> /isa/BA5
- J2 pad 58: BA4 -> /isa/BA4
- J2 pad 59: BA3 -> /isa/BA3
- J2 pad 60: BA2 -> /isa/BA2
- J2 pad 61: BA1 -> /isa/BA1
- J2 pad 62: BA0 -> /isa/BA0
- J2 pad 82: BA23 -> /isa/BA23
- J2 pad 83: BA22 -> /isa/BA22
- J2 pad 84: BA21 -> /isa/BA21
- J2 pad 85: BA20 -> /isa/BA20
- J2 pad 86: BA19 -> /isa/BA19
- J2 pad 87: BA18 -> /isa/BA18
- J2 pad 88: BA17 -> /isa/BA17
- J2 pad 91: BD24 -> /isa/BD8
- J2 pad 92: BD25 -> /isa/BD9
- J2 pad 93: BD26 -> /isa/BD10
- J2 pad 94: BD27 -> /isa/BD11
- J2 pad 95: BD28 -> /isa/BD12
- J2 pad 96: BD29 -> /isa/BD13
- J2 pad 97: BD30 -> /isa/BD14
- J2 pad 98: BD31 -> /isa/BD15
- J3 pad 32: unconnected-(J3-IO-Pad32) -> /isa/~{IOCHCK}
- J3 pad 33: BD23 -> /isa/BD7
- J3 pad 34: BD22 -> /isa/BD6
- J3 pad 35: BD21 -> /isa/BD5
- J3 pad 36: BD20 -> /isa/BD4
- J3 pad 37: BD19 -> /isa/BD3
- J3 pad 38: BD18 -> /isa/BD2
- J3 pad 39: BD17 -> /isa/BD1
- J3 pad 40: BD16 -> /isa/BD0
- J3 pad 43: BA19 -> /isa/BA19
- J3 pad 44: BA18 -> /isa/BA18
- J3 pad 45: BA17 -> /isa/BA17
- J3 pad 46: BA16 -> /isa/BA16
- J3 pad 47: BA15 -> /isa/BA15
- J3 pad 48: BA14 -> /isa/BA14
- J3 pad 49: BA13 -> /isa/BA13
- J3 pad 50: BA12 -> /isa/BA12
- J3 pad 51: BA11 -> /isa/BA11
- J3 pad 52: BA10 -> /isa/BA10
- J3 pad 53: BA9 -> /isa/BA9
- J3 pad 54: BA8 -> /isa/BA8
- J3 pad 55: BA7 -> /isa/BA7
- J3 pad 56: BA6 -> /isa/BA6
- J3 pad 57: BA5 -> /isa/BA5
- J3 pad 58: BA4 -> /isa/BA4
- J3 pad 59: BA3 -> /isa/BA3
- J3 pad 60: BA2 -> /isa/BA2
- J3 pad 61: BA1 -> /isa/BA1
- J3 pad 62: BA0 -> /isa/BA0
- J3 pad 82: BA23 -> /isa/BA23
- J3 pad 83: BA22 -> /isa/BA22
- J3 pad 84: BA21 -> /isa/BA21
- J3 pad 85: BA20 -> /isa/BA20
- J3 pad 86: BA19 -> /isa/BA19
- J3 pad 87: BA18 -> /isa/BA18
- J3 pad 88: BA17 -> /isa/BA17
- J3 pad 91: BD24 -> /isa/BD8
- J3 pad 92: BD25 -> /isa/BD9
- J3 pad 93: BD26 -> /isa/BD10
- J3 pad 94: BD27 -> /isa/BD11
- J3 pad 95: BD28 -> /isa/BD12
- J3 pad 96: BD29 -> /isa/BD13
- J3 pad 97: BD30 -> /isa/BD14
- J3 pad 98: BD31 -> /isa/BD15
- L1 pad 1: Net-(J13-Pin_4) -> +5V
- L1 pad 2: /audio/PINK_TIP -> /audio/PWR1
- L2 pad 1: Net-(J13-Pin_2) -> Net-(J13-Pin_4)
- L2 pad 2: /audio/PINK_RING -> /audio/PINK_TIP
- L3 pad 1: Net-(C101-Pad2) -> Net-(J13-Pin_2)
- L3 pad 2: /audio/BLUE_TIP -> /audio/PINK_RING
- L4 pad 1: Net-(C102-Pad2) -> Net-(C54-Pad2)
- L4 pad 2: /audio/BLUE_RING -> /audio/BLUE_TIP
- R10 pad 1: Net-(C93-Pad1) -> Net-(U27B-+)
- R10 pad 2: Net-(U54B--) -> /audio/VREF
- R11 pad 1: Net-(U54B--) -> Net-(C51-Pad1)
- R11 pad 2: Net-(C92-Pad2) -> Net-(U27B--)
- R12 pad 1: Net-(J13-Pin_4) -> Net-(J13-Pin_2)
- R13 pad 1: Net-(J13-Pin_2) -> Net-(J13-Pin_4)
- R14 pad 1: +5VA -> Net-(U27B--)
- R14 pad 2: Net-(J13-Pin_1) -> Net-(C50-Pad2)
- R15 pad 1: Net-(C101-Pad1) -> Net-(U28A--)
- R15 pad 2: Net-(U55A--) -> Net-(C53-Pad2)
- R16 pad 1: Net-(C102-Pad1) -> Net-(C54-Pad1)
- R16 pad 2: Net-(U55B--) -> Net-(U28A--)
- R17 pad 1: Net-(U55A-+) -> Net-(U28A-+)
- R18 pad 1: Net-(U55A--) -> Net-(C59-Pad1)
- R18 pad 2: Net-(C96-Pad2) -> Net-(U28B--)
- R19 pad 1: Net-(U55B--) -> Net-(U28B--)
- R19 pad 2: Net-(C103-Pad2) -> Net-(C58-Pad2)
- R6 pad 1: Net-(U54A--) -> Net-(C45-Pad1)
- R6 pad 2: Net-(C89-Pad2) -> Net-(U27A--)
- R7 pad 1: Net-(C91-Pad1) -> Net-(U27A--)
- R7 pad 2: Net-(U54A--) -> Net-(C44-Pad2)
- R8 pad 2: Net-(U54A-+) -> Net-(U27A-+)
- R9 pad 1: Net-(U54B-+) -> +5VA
- R9 pad 2: /audio/VREF -> Net-(J13-Pin_1)
- RN1 pad 2: /cpu/~{MMUDIS} -> ~{HALT}
- RN1 pad 3: /cpu/~{CDIS} -> ~{BERR}
- RN1 pad 4: ~{IPL2} -> ~{STERM}
- RN1 pad 5: ~{BGACK} -> ~{DSACK1}
- RN1 pad 6: ~{HALT} -> ~{DSACK0}
- RN1 pad 7: ~{DSACK1} -> ~{AVEC}
- RN1 pad 8: ~{BR} -> ~{BGACK}
- RN1 pad 9: ~{BERR} -> ~{BR}
- RN10 pad 2: /dmac1/~{DRQ1} -> ~{DRQ1}
- RN10 pad 3: /dmac1/~{DTC} -> /dmac/~{DTC}
- RN10 pad 4: /dmac1/~{DACK0} -> ~{DACK0}
- RN10 pad 5: /dmac1/~{DACK1} -> ~{DACK1}
- RN11 pad 2: /dmac0/~{OWN} -> ~{DRQ2}
- RN11 pad 3: /dmac0/~{HIBYTE} -> ~{DRQ3}
- RN11 pad 4: /dmac0/~{UAS} -> ~{DACK2}
- RN11 pad 5: /dmac0/~{DBEN} -> ~{DACK3}
- RN2 pad 3: ~{IPL0} -> ~{CIIN}
- RN2 pad 4: ~{IPL1} -> ~{CBACK}
- RN2 pad 5: ~{AVEC} -> ~{CDIS}
- RN2 pad 6: ~{DSACK0} -> ~{IPL0}
- RN2 pad 7: ~{STERM} -> ~{IPL2}
- RN2 pad 8: ~{CBACK} -> ~{IPL1}
- RN2 pad 9: ~{CIIN} -> ~{MMUDIS}
- RN3 pad 1: /dram/~{CAS0} -> +5V
- RN3 pad 2: /dram/~{CAS2} -> /isa/~{DACK7}
- RN3 pad 3: /dram/~{CAS3} -> /isa/~{DACK6}
- RN3 pad 4: /dram/~{CAS1} -> /isa/~{DACK5}
- RN3 pad 5: Net-(RN3-R4.2) -> /isa/~{DACK0}
- RN3 pad 6: Net-(RN3-R3.2) -> /isa/~{DACK2}
- RN3 pad 7: Net-(RN3-R2.2) -> /isa/~{REFRESH}
- RN3 pad 8: Net-(RN3-R1.2) -> /isa/~{DACK1}
- RN4 pad 1: /dram/~{RAS3} -> GND
- RN4 pad 2: /dram/~{RAS2} -> /isa/DRQ7
- RN4 pad 3: /dram/~{RAS1} -> /isa/DRQ6
- RN4 pad 4: /dram/~{RAS0} -> /isa/DRQ5
- RN4 pad 5: Net-(RN4-R4.2) -> /isa/DRQ0
- RN4 pad 6: Net-(RN4-R3.2) -> /isa/DRQ1
- RN4 pad 7: Net-(RN4-R2.2) -> /isa/DRQ2
- RN4 pad 8: Net-(RN4-R1.2) -> /isa/DRQ3
- RN5 pad 1: +5V -> GND
- RN5 pad 2: /isa/~{DACK7} -> IRQ3
- RN5 pad 3: /isa/~{DACK6} -> IRQ4
- RN5 pad 4: /isa/~{DACK5} -> IRQ5
- RN5 pad 5: /isa/~{DACK0} -> IRQ6
- RN5 pad 6: /isa/~{DACK2} -> IRQ7
- RN5 pad 7: /isa/~{REFRESH} -> IRQ2
- RN6 pad 2: /isa/DRQ7 -> IRQ14
- RN6 pad 3: /isa/DRQ6 -> IRQ15
- RN6 pad 4: /isa/DRQ5 -> IRQ12
- RN6 pad 5: /isa/DRQ0 -> IRQ11
- RN6 pad 6: /isa/DRQ1 -> IRQ10
- RN6 pad 7: /isa/DRQ2 -> unconnected-(RN6-R6-Pad7)
- RN7 pad 1: GND -> +5V
- RN7 pad 2: IRQ3 -> /timer_irqc/~{IRQ0}
- RN7 pad 3: IRQ4 -> /timer_irqc/~{IRQ1}
- RN7 pad 4: IRQ5 -> ~{MFP_IRQ}
- RN7 pad 5: IRQ6 -> AUDIO_IRQ
- RN7 pad 6: IRQ7 -> ~{DMAC1_IRQ}
- RN7 pad 7: IRQ2 -> ~{DMAC0_IRQ}
- RN8 pad 1: GND -> Net-(RN8-R1.1)
- RN8 pad 2: IRQ14 -> Net-(RN8-R2.1)
- RN8 pad 3: IRQ15 -> Net-(RN8-R3.1)
- RN8 pad 4: IRQ12 -> Net-(RN8-R4.1)
- RN8 pad 5: IRQ11 -> Net-(J11-Pin_9)
- RN8 pad 6: IRQ10 -> Net-(J11-Pin_7)
- RN8 pad 7: unconnected-(RN8-R6-Pad7) -> Net-(J11-Pin_5)
- RN9 pad 2: /dmac1/~{OWN} -> /dmac/~{OWN}
- RN9 pad 3: /dmac1/~{HIBYTE} -> /dmac/~{HIBYTE}
- RN9 pad 4: /dmac1/~{UAS} -> /dmac/~{UAS}
- RN9 pad 5: /dmac1/~{DBEN} -> /dmac/~{DBEN}
- RN9 pad 6: /dmac1/~{DDIR} -> /dmac/~{DDIR}
- RN9 pad 7: /dmac1/~{DRQ0} -> ~{DRQ0}
- U1 pad B1: /cpu/~{RMC} -> unconnected-(U1A-~{RMC}-PadB1)
- U1 pad D3: /cpu/~{OCS} -> unconnected-(U1A-~{OCS}-PadD3)
- U1 pad F13: /cpu/~{MMUDIS} -> ~{MMUDIS}
- U1 pad H12: /cpu/~{CDIS} -> ~{CDIS}
- U1 pad J13: /cpu/~{REFILL} -> unconnected-(U1A-~{REFILL}-PadJ13)
- U1 pad M1: /cpu/~{DBEN} -> unconnected-(U1A-~{DBEN}-PadM1)
- U1 pad M2: /cpu/~{ECS} -> unconnected-(U1A-~{ECS}-PadM2)
- U10 pad 1: +5V -> Net-(U38A-O0)
- U10 pad 10: A14 -> ~{DS}
- U10 pad 11: A3 -> unconnected-(U10-Pad11)
- U10 pad 12: A15 -> unconnected-(U10-Pad12)
- U10 pad 13: A4 -> unconnected-(U10-Pad13)
- U10 pad 14: A16 -> +5V
- U10 pad 2: MA7 -> /dmac/~{RETRY}
- U10 pad 3: GND -> Net-(U10-Pad3)
- U10 pad 4: MA8 -> (no net)
- U10 pad 5: MA9 -> (no net)
- U10 pad 6: MA10 -> (no net)
- U10 pad 7: MA11 -> GND
- U10 pad 8: A13 -> Net-(U11-~{CS})
- U10 pad 9: A2 -> ~{DUART_CS}
- U11 pad 1: R/~{W} -> BA0
- U11 pad 10: GND -> /serial/RxDB
- U11 pad 11: D12 -> /serial/TxDB
- U11 pad 12: D31 -> /serial/~{RTSB}
- U11 pad 13: D13 -> unconnected-(U11-OP3-Pad13)
- U11 pad 14: D30 -> unconnected-(U11-OP5-Pad14)
- U11 pad 15: D14 -> unconnected-(U11-OP7-Pad15)
- U11 pad 16: D29 -> BD25
- U11 pad 17: D28 -> BD27
- U11 pad 18: D15 -> BD29
- U11 pad 19: GND -> BD31
- U11 pad 2: MD12 -> unconnected-(U11-IP3-Pad2)
- U11 pad 20: +5V -> GND
- U11 pad 3: MD28 -> BA1
- U11 pad 4: MD29 -> /serial/~{CTSB}
- U11 pad 5: MD13 -> BA2
- U11 pad 6: MD30 -> BA3
- U11 pad 7: MD14 -> /serial/~{CTSA}
- U11 pad 8: MD31 -> R/~{W}
- U11 pad 9: MD15 -> ~{DSACK0}
- U12 pad 1: 8MHz -> Net-(U12-C1+)
- U12 pad 10: GND -> /serial/~{RTSB}
- U12 pad 11: /isa/IOCHRDY -> /serial/TxDB
- U12 pad 12: /isa/~{MEMW} -> /serial/RxDB
- U12 pad 13: /isa/~{MEMR} -> /serial/RxDP2
- U12 pad 14: /isa/~{IOW} -> /serial/TxDP2
- U12 pad 15: /isa/~{IOR} -> GND
- U12 pad 16: /isa/~{SMEMW} -> +5V
- U12 pad 2: ~{ISAMEMSEL} -> Net-(U12-VS+)
- U12 pad 3: ~{ISAIOSEL} -> Net-(U12-C1-)
- U12 pad 4: ~{AS} -> Net-(U12-C2+)
- U12 pad 5: ~{DS} -> Net-(U12-C2-)
- U12 pad 6: R/~{W} -> Net-(U12-VS-)
- U12 pad 7: /isa/~{MEMCS16} -> /serial/~{RTSP2}
- U12 pad 8: /isa/~{IOCS16} -> /serial/~{CTSP2}
- U12 pad 9: /isa/~{NOWS} -> /serial/~{CTSB}
- U13 pad 1: 8MHz -> /floppy/WP
- U13 pad 10: GND -> BA2
- U13 pad 11: /isa/IOCHRDY -> BD24
- U13 pad 12: unconnected-(U13-IO8-Pad12) -> GND
- U13 pad 13: unconnected-(U13-IO7-Pad13) -> BD25
- U13 pad 14: unconnected-(U13-IO6-Pad14) -> BD26
- U13 pad 15: unconnected-(U13-IO5-Pad15) -> BD27
- U13 pad 16: unconnected-(U13-IO4-Pad16) -> GND
- U13 pad 17: unconnected-(U13-I03-Pad17) -> BD28
- U13 pad 18: ~{DSACK1} -> +5V
- U13 pad 19: ~{DSACK0} -> BD29
- U13 pad 2: ~{ISAMEMSEL} -> /floppy/TRK0
- U13 pad 20: +5V -> BD30
- U13 pad 3: ~{ISAIOSEL} -> unconnected-(U13-~{DACK}-Pad3)
- U13 pad 4: ~{AS} -> ~{RD}
- U13 pad 5: ~{DS} -> ~{WR}
- U13 pad 6: R/~{W} -> ~{FDC_CS}
- U13 pad 7: /isa/~{MEMCS16} -> BA0
- U13 pad 8: /isa/~{IOCS16} -> BA1
- U13 pad 9: /isa/~{NOWS} -> GND
- U14 pad 1: +5V -> unconnected-(U14-TEST0-Pad1)
- U14 pad 10: GND -> ~{WR}
- U14 pad 11: BA7 -> unconnected-(U14-SYNC-Pad11)
- U14 pad 12: BA6 -> /i8242/BD24
- U14 pad 13: BA5 -> /i8242/BD25
- U14 pad 14: BA4 -> /i8242/BD26
- U14 pad 15: BA3 -> /i8242/BD27
- U14 pad 16: BA2 -> /i8242/BD28
- U14 pad 17: BA1 -> /i8242/BD29
- U14 pad 18: BA0 -> /i8242/BD30
- U14 pad 19: GND -> /i8242/BD31
- U14 pad 2: A0 -> GND
- U14 pad 20: +5V -> GND
- U14 pad 3: A1 -> 8MHz
- U14 pad 4: A2 -> ~{RST}
- U14 pad 5: A3 -> unconnected-(U14-TH_SS-Pad5)
- U14 pad 6: A4 -> ~{I8242_CS}
- U14 pad 7: A5 -> unconnected-(U14-TL_EA-Pad7)
- U14 pad 8: A6 -> ~{RD}
- U14 pad 9: A7 -> /i8242/BA0
- U15 pad 1: +5V -> GND
- U15 pad 10: GND -> Net-(U15-CAP)
- U15 pad 11: BA23 -> FREQ_SEL0
- U15 pad 12: BA22 -> FREQ_SEL1
- U15 pad 13: BA21 -> FREQ_SEL2
- U15 pad 14: BA20 -> +5V
- U15 pad 2: A16 -> unconnected-(U15-XO-Pad2)
- U15 pad 3: A17 -> unconnected-(U15-XI-Pad3)
- U15 pad 4: A18 -> 14.31818MHz
- U15 pad 5: A19 -> 24MHz
- U15 pad 6: A20 -> unconnected-(U15-~{LOP}-Pad6)
- U15 pad 7: A21 -> GND
- U15 pad 8: A22 -> PROC_CLK
- U15 pad 9: A23 -> +5V
- U16 pad 1: +5V -> /power/BUZ+
- U16 pad 10: GND -> /power/~{PSW}
- U16 pad 11: BA15 -> GND
- U16 pad 12: BA14 -> GND
- U16 pad 2: A8 -> Net-(U16D-HDD+)
- U16 pad 3: A9 -> (no net)
- U16 pad 4: A10 -> Net-(U16D-HDD-)
- U16 pad 5: A11 -> (no net)
- U16 pad 6: A12 -> +5V
- U16 pad 7: A13 -> Net-(U16C-BUZ-)
- U16 pad 8: A14 -> Net-(U16E-PWR-)
- U16 pad 9: A15 -> ~{RST}
- U17 pad 1: +5V -> (no net)
- U17 pad 10: GND -> (no net)
- U17 pad 11: BA31 -> (no net)
- U17 pad 12: BA30 -> (no net)
- U17 pad 13: BA29 -> (no net)
- U17 pad 14: BA28 -> (no net)
- U17 pad 2: A24 -> (no net)
- U17 pad 3: A25 -> ~{HDDLED}
- U17 pad 4: A26 -> Net-(U16D-HDD+)
- U17 pad 5: A27 -> (no net)
- U17 pad 6: A28 -> (no net)
- U17 pad 7: A29 -> (no net)
- U17 pad 8: A30 -> (no net)
- U17 pad 9: A31 -> (no net)
- U22 pad 1: /floppy/WP -> R/~{W}
- U22 pad 10: BA2 -> unconnected-(U22-RC-Pad10)
- U22 pad 11: BD24 -> +5V
- U22 pad 12: GND -> unconnected-(U22-NC-Pad12)
- U22 pad 13: BD25 -> unconnected-(U22-TAO-Pad13)
- U22 pad 14: BD26 -> unconnected-(U22-TBO-Pad14)
- U22 pad 15: BD27 -> unconnected-(U22-TCO-Pad15)
- U22 pad 16: GND -> unconnected-(U22-TDO-Pad16)
- U22 pad 17: BD28 -> 3.6864MHz
- U22 pad 18: +5V -> unconnected-(U22-XTAL2-Pad18)
- U22 pad 19: BD29 -> unconnected-(U22-TAI-Pad19)
- U22 pad 2: /floppy/TRK0 -> BA0
- U22 pad 20: BD30 -> unconnected-(U22-TBI-Pad20)
- U22 pad 21: GND -> ~{RST}
- U22 pad 22: BD31 -> IRQ7
- U22 pad 23: FDC_IRQ -> IRQ6
- U22 pad 24: FDC_DRQ -> IRQ5
- U22 pad 25: FDC_TC -> IRQ4
- U22 pad 26: /floppy/~{INDEX} -> IRQ3
- U22 pad 27: +5V -> ~{DUART_IRQ}
- U22 pad 28: /floppy/DRATE0 -> MS_IRQ
- U22 pad 29: unconnected-(U22-DRATE1-Pad29) -> KB_IRQ
- U22 pad 3: ~{FDC_DACK} -> BA1
- U22 pad 31: /floppy/DSKCHG -> unconnected-(U22-~{RR}-Pad31)
- U22 pad 32: RST -> ~{MFP_IRQ}
- U22 pad 33: 24MHz -> unconnected-(U22-~{IEO}-Pad33)
- U22 pad 34: unconnected-(U22-XTAL2-Pad34) -> /timer_irqc/~{IEO0}
- U22 pad 35: /floppy/INVERT -> 4MHz
- U22 pad 37: unconnected-(U22-LOFIL-Pad37) -> BD24
- U22 pad 38: unconnected-(U22-HIFIL-Pad38) -> BD25
- U22 pad 39: unconnected-(U22-PLL0-Pad39) -> BD26
- U22 pad 4: ~{RD} -> BA2
- U22 pad 40: unconnected-(U22-PLL1-Pad40) -> BD27
- U22 pad 41: /floppy/RDATA -> BD28
- U22 pad 42: unconnected-(U22-NC-Pad42) -> BD29
- U22 pad 43: unconnected-(U22-NC-Pad43) -> BD30
- U22 pad 44: unconnected-(U22-NC-Pad44) -> BD31
- U22 pad 45: GND -> unconnected-(U22-~{IACK}-Pad45)
- U22 pad 46: +5V -> ~{DSACK0}
- U22 pad 47: unconnected-(U22-NC-Pad47) -> ~{DS}
- U22 pad 48: unconnected-(U22-MFM-Pad48) -> ~{MFP1_CS}
- U22 pad 5: ~{WR} -> BA3
- U22 pad 6: ~{FDC_CS} -> BA4
- U22 pad 7: BA0 -> unconnected-(U22-TC-Pad7)
- U22 pad 8: BA1 -> unconnected-(U22-SO-Pad8)
- U22 pad 9: GND -> unconnected-(U22-SI-Pad9)
- U23 pad 1: unconnected-(U23-TEST0-Pad1) -> ~{AS}
- U23 pad 10: ~{WR} -> GND
- U23 pad 12: BD24 -> unconnected-(U23-IO8-Pad12)
- U23 pad 13: BD25 -> unconnected-(U23-IO7-Pad13)
- U23 pad 14: BD26 -> ~{WR}
- U23 pad 15: BD27 -> ~{RD}
- U23 pad 16: BD28 -> ~{BYTE3}
- U23 pad 17: BD29 -> ~{BYTE2}
- U23 pad 18: BD30 -> ~{BYTE1}
- U23 pad 19: BD31 -> ~{BYTE0}
- U23 pad 2: unconnected-(U23-XTAL1-Pad2) -> ~{DS}
- U23 pad 20: GND -> +5V
- U23 pad 3: unconnected-(U23-XTAL2-Pad3) -> R/~{W}
- U23 pad 4: ~{RST} -> SIZ0
- U23 pad 5: unconnected-(U23-TH_SS-Pad5) -> SIZ1
- U23 pad 6: ~{I8242_CS} -> A0
- U23 pad 7: unconnected-(U23-TL_EA-Pad7) -> A1
- U23 pad 8: ~{RD} -> unconnected-(U23-I8-Pad8)
- U23 pad 9: BA0 -> unconnected-(U23-I9-Pad9)
- U29 pad 1: R/~{W} -> A0
- U29 pad 10: GND -> unconnected-(U29A-GND-Pad10)
- U29 pad 11: D31 -> unconnected-(U29A-VCCINT-Pad11)
- U29 pad 12: D30 -> unconnected-(U29A-VCCIO-Pad12)
- U29 pad 13: D29 -> A8
- U29 pad 14: D28 -> A9
- U29 pad 15: D27 -> A10
- U29 pad 16: D26 -> A11
- U29 pad 17: D25 -> A12
- U29 pad 18: D24 -> A13
- U29 pad 19: /dmac1/~{HIBYTE} -> A14
- U29 pad 2: D16 -> A1
- U29 pad 20: +5V -> A15
- U29 pad 3: D17 -> A2
- U29 pad 4: D18 -> A3
- U29 pad 5: D19 -> A4
- U29 pad 6: D20 -> A5
- U29 pad 7: D21 -> A6
- U29 pad 8: D22 -> A7
- U29 pad 9: D23 -> unconnected-(U29B-~{CE}-Pad9)
- U30 pad 1: /dmac1/~{DDIR} -> unconnected-(U30-OE-Pad1)
- U30 pad 10: GND -> unconnected-(U30-GND-Pad10)
- U30 pad 11: D23 -> unconnected-(U30-Load-Pad11)
- U30 pad 12: D22 -> /isa/BA0
- U30 pad 13: D21 -> /isa/BA1
- U30 pad 14: D20 -> /isa/BA2
- U30 pad 15: D19 -> /isa/BA3
- U30 pad 16: D18 -> /isa/BA4
- U30 pad 17: D17 -> /isa/BA5
- U30 pad 18: D16 -> /isa/BA6
- U30 pad 19: /dmac1/~{DBEN} -> /isa/BA7
- U30 pad 2: /dmac1/A8/D0 -> A7
- U30 pad 20: +5V -> unconnected-(U30-VCC-Pad20)
- U30 pad 3: /dmac1/A9/D1 -> A6
- U30 pad 4: /dmac1/A10/D2 -> A5
- U30 pad 5: /dmac1/A11/D3 -> A4
- U30 pad 6: /dmac1/A12/D4 -> A3
- U30 pad 7: /dmac1/A13/D5 -> A2
- U30 pad 8: /dmac1/A14/D6 -> A1
- U30 pad 9: /dmac1/A15/D7 -> A0
- U31 pad 1: /dmac1/~{OWN} -> unconnected-(U31-A->B-Pad1)
- U31 pad 10: GND -> unconnected-(U31-GND-Pad10)
- U31 pad 11: /dmac1/UAS -> /isa/BD0
- U31 pad 12: A15 -> /isa/BD1
- U31 pad 13: A14 -> /isa/BD2
- U31 pad 14: A13 -> /isa/BD3
- U31 pad 15: A12 -> /isa/BD4
- U31 pad 16: A11 -> /isa/BD5
- U31 pad 17: A10 -> /isa/BD6
- U31 pad 18: A9 -> /isa/BD7
- U31 pad 19: A8 -> unconnected-(U31-CE-Pad19)
- U31 pad 2: /dmac1/A8/D0 -> D23
- U31 pad 20: +5V -> unconnected-(U31-VCC-Pad20)
- U31 pad 3: /dmac1/A9/D1 -> D22
- U31 pad 4: /dmac1/A10/D2 -> D21
- U31 pad 5: /dmac1/A11/D3 -> D20
- U31 pad 6: /dmac1/A12/D4 -> D19
- U31 pad 7: /dmac1/A13/D5 -> D18
- U31 pad 8: /dmac1/A14/D6 -> D17
- U31 pad 9: /dmac1/A15/D7 -> D16
- U32 pad 1: /dmac1/~{DDIR} -> unconnected-(U32-A->B-Pad1)
- U32 pad 10: /dmac1/PCL0 -> unconnected-(U32-GND-Pad10)
- U32 pad 11: ~{BGACK} -> /isa/BD15
- U32 pad 12: /dmac1/~{DTC} -> /isa/BD14
- U32 pad 13: unconnected-(U32-~{DTACK}-Pad13) -> /isa/BD13
- U32 pad 14: A0 -> /isa/BD12
- U32 pad 15: ~{DS} -> /isa/BD11
- U32 pad 16: ~{AS} -> /isa/BD10
- U32 pad 17: R/~{W} -> /isa/BD9
- U32 pad 18: GND -> /isa/BD8
- U32 pad 19: ~{DMAC1_CS} -> unconnected-(U32-CE-Pad19)
- U32 pad 2: A25 -> D24
- U32 pad 20: +5V -> unconnected-(U32-VCC-Pad20)
- U32 pad 3: A26 -> D25
- U32 pad 4: A27 -> D26
- U32 pad 5: /dmac1/~{DRQ1} -> D27
- U32 pad 6: /dmac1/~{DRQ0} -> D28
- U32 pad 7: A28 -> D29
- U32 pad 8: A29 -> D30
- U32 pad 9: /dmac1/PCL1 -> D31
- U33 pad 1: /dmac1/~{DDIR} -> unconnected-(U33-OE-Pad1)
- U33 pad 10: GND -> unconnected-(U33-GND-Pad10)
- U33 pad 11: D31 -> unconnected-(U33-Load-Pad11)
- U33 pad 12: D30 -> /isa/BA8
- U33 pad 13: D29 -> /isa/BA9
- U33 pad 14: D28 -> /isa/BA10
- U33 pad 15: D27 -> /isa/BA11
- U33 pad 16: D26 -> /isa/BA12
- U33 pad 17: D25 -> /isa/BA13
- U33 pad 18: D24 -> /isa/BA14
- U33 pad 19: /dmac1/~{DBEN} -> /isa/BA15
- U33 pad 2: /dmac1/A16/D8 -> A15
- U33 pad 20: +5V -> unconnected-(U33-VCC-Pad20)
- U33 pad 3: /dmac1/A17/D9 -> A14
- U33 pad 4: /dmac1/A18/D10 -> A13
- U33 pad 5: /dmac1/A19/D11 -> A12
- U33 pad 6: /dmac1/A20/D12 -> A11
- U33 pad 7: /dmac1/A21/D13 -> A10
- U33 pad 8: /dmac1/A22/D14 -> A9
- U33 pad 9: /dmac1/A23/D15 -> A8
- U34 pad 1: /dmac1/~{OWN} -> unconnected-(U34-OE-Pad1)
- U34 pad 10: GND -> unconnected-(U34-GND-Pad10)
- U34 pad 11: /dmac1/UAS -> unconnected-(U34-Load-Pad11)
- U34 pad 12: A23 -> /isa/BA16
- U34 pad 13: A22 -> /isa/BA17
- U34 pad 14: A21 -> /isa/BA18
- U34 pad 15: A20 -> /isa/BA19
- U34 pad 16: A19 -> /isa/BA20
- U34 pad 17: A18 -> /isa/BA21
- U34 pad 18: A17 -> /isa/BA22
- U34 pad 19: A16 -> /isa/BA23
- U34 pad 2: /dmac1/A16/D8 -> A23
- U34 pad 20: +5V -> unconnected-(U34-VCC-Pad20)
- U34 pad 3: /dmac1/A17/D9 -> A22
- U34 pad 4: /dmac1/A18/D10 -> A21
- U34 pad 5: /dmac1/A19/D11 -> A20
- U34 pad 6: /dmac1/A20/D12 -> A19
- U34 pad 7: /dmac1/A21/D13 -> A18
- U34 pad 8: /dmac1/A22/D14 -> A17
- U34 pad 9: /dmac1/A23/D15 -> A16
- U35 pad 1: Net-(U36B-O0) -> +5V
- U35 pad 10: /dmac0/~{RETRY0} -> +5V
- U35 pad 11: /dmac0/~{RETRY0} -> ~{HALT}
- U35 pad 12: Net-(U35-Pad12) -> ~{BERR}
- U35 pad 13: Net-(U36A-O3) -> /dmac/~{RETRY}
- U35 pad 14: +5V -> unconnected-(U35-GS-Pad14)
- U35 pad 2: Net-(U35-Pad2) -> +5V
- U35 pad 3: /dmac1/~{RETRY1} -> +5V
- U35 pad 4: /dmac1/~{RETRY1} -> ~{RST}
- U35 pad 5: Net-(U36B-O3) -> GND
- U35 pad 6: Net-(U35-Pad2) -> /dmac/~{BEC2}
- U35 pad 7: GND -> /dmac/~{BEC1}
- U35 pad 8: Net-(U35-Pad12) -> GND
- U35 pad 9: Net-(U36A-O0) -> /dmac/~{BEC0}
- U36 pad 1: GND -> /dmac/~{DDIR}
- U36 pad 10: /dmac1/~{HALT1} -> PCL2
- U36 pad 11: /dmac1/~{BERR1} -> ~{BGACK}
- U36 pad 12: Net-(U36B-O0) -> /dmac/~{DTC}
- U36 pad 13: ~{BERR} -> unconnected-(U36-~{DTACK}-Pad13)
- U36 pad 14: ~{HALT} -> /dmac/A0
- U36 pad 15: GND -> ~{DS}
- U36 pad 16: +5V -> ~{AS}
- U36 pad 2: ~{HALT} -> /dmac/A25
- U36 pad 3: ~{BERR} -> /dmac/A26
- U36 pad 4: Net-(U36A-O0) -> /dmac/A27
- U36 pad 5: /dmac0/~{BERR0} -> ~{DRQ3}
- U36 pad 6: /dmac0/~{HALT0} -> ~{DRQ2}
- U36 pad 7: Net-(U36A-O3) -> /dmac/A28
- U36 pad 8: GND -> /dmac/A29
- U36 pad 9: Net-(U36B-O3) -> PCL3
- U37 pad 1: +5V -> /dmac/~{DDIR}
- U37 pad 10: +5V -> PCL0
- U37 pad 11: /dmac1/~{HALT1} -> ~{BGACK}
- U37 pad 12: /dmac1/~{BERR1} -> /dmac/~{DTC}
- U37 pad 13: /dmac1/~{RETRY1} -> unconnected-(U37-~{DTACK}-Pad13)
- U37 pad 14: unconnected-(U37-GS-Pad14) -> /dmac/A0
- U37 pad 15: unconnected-(U37-EO-Pad15) -> ~{DS}
- U37 pad 16: +5V -> ~{AS}
- U37 pad 2: +5V -> /dmac/A25
- U37 pad 3: +5V -> /dmac/A26
- U37 pad 4: ~{RST} -> /dmac/A27
- U37 pad 5: GND -> ~{DRQ1}
- U37 pad 6: /dmac1/~{BEC2} -> ~{DRQ0}
- U37 pad 7: /dmac1/~{BEC1} -> /dmac/A28
- U37 pad 8: GND -> /dmac/A29
- U37 pad 9: /dmac1/~{BEC0} -> PCL1
- U38 pad 1: R/~{W} -> GND
- U38 pad 10: GND -> unconnected-(U38B-O2-Pad10)
- U38 pad 11: D31 -> unconnected-(U38B-O1-Pad11)
- U38 pad 12: D30 -> unconnected-(U38B-O0-Pad12)
- U38 pad 13: D29 -> unconnected-(U38B-A1-Pad13)
- U38 pad 14: D28 -> unconnected-(U38B-A0-Pad14)
- U38 pad 15: D27 -> unconnected-(U38B-E-Pad15)
- U38 pad 16: D26 -> +5V
- U38 pad 2: D16 -> ~{HALT}
- U38 pad 3: D17 -> ~{BERR}
- U38 pad 4: D18 -> Net-(U38A-O0)
- U38 pad 5: D19 -> ~{BERR}
- U38 pad 6: D20 -> ~{HALT}
- U38 pad 7: D21 -> Net-(U38A-O3)
- U38 pad 8: D22 -> GND
- U38 pad 9: D23 -> unconnected-(U38B-O3-Pad9)
- U40 pad 1: /dmac0/~{OWN} -> /dmac/~{UAS}
- U40 pad 10: GND -> unconnected-(U40-Pad10)
- U40 pad 11: /dmac0/UAS -> unconnected-(U40-Pad11)
- U40 pad 12: A15 -> unconnected-(U40-Pad12)
- U40 pad 13: A14 -> unconnected-(U40-Pad13)
- U40 pad 14: A13 -> +5V
- U40 pad 2: /dmac0/A8/D0 -> /dmac/UAS
- U40 pad 3: /dmac0/A9/D1 -> unconnected-(U40-Pad3)
- U40 pad 4: /dmac0/A10/D2 -> unconnected-(U40-Pad4)
- U40 pad 5: /dmac0/A11/D3 -> unconnected-(U40-Pad5)
- U40 pad 6: /dmac0/A12/D4 -> unconnected-(U40-Pad6)
- U40 pad 7: /dmac0/A13/D5 -> GND
- U40 pad 8: /dmac0/A14/D6 -> unconnected-(U40-Pad8)
- U40 pad 9: /dmac0/A15/D7 -> unconnected-(U40-Pad9)
- U41 pad 1: /dmac0/~{DDIR} -> R/~{W}
- U41 pad 10: FDC_TC -> GND
- U41 pad 11: ~{BGACK} -> D31
- U41 pad 12: /dmac0/~{DTC} -> D30
- U41 pad 13: unconnected-(U41-~{DTACK}-Pad13) -> D29
- U41 pad 14: A0 -> D28
- U41 pad 15: ~{DS} -> D27
- U41 pad 16: ~{AS} -> D26
- U41 pad 17: R/~{W} -> D25
- U41 pad 18: GND -> D24
- U41 pad 19: ~{DMAC0_CS} -> /dmac/demuxer/~{HIBYTE}
- U41 pad 2: A25 -> D16
- U41 pad 3: A26 -> D17
- U41 pad 4: A27 -> D18
- U41 pad 5: /dmac0/~{DRQ1} -> D19
- U41 pad 6: /dmac0/~{DRQ0} -> D20
- U41 pad 7: A28 -> D21
- U41 pad 8: A29 -> D22
- U41 pad 9: /dmac0/PCL1 -> D23
- U42 pad 1: /dmac0/~{DDIR} -> /dmac/demuxer/~{DDIR}
- U42 pad 11: D31 -> D23
- U42 pad 12: D30 -> D22
- U42 pad 13: D29 -> D21
- U42 pad 14: D28 -> D20
- U42 pad 15: D27 -> D19
- U42 pad 16: D26 -> D18
- U42 pad 17: D25 -> D17
- U42 pad 18: D24 -> D16
- U42 pad 19: /dmac0/~{DBEN} -> /dmac/demuxer/~{DBEN}
- U42 pad 2: /dmac0/A16/D8 -> /dmac/MUX0
- U42 pad 3: /dmac0/A17/D9 -> /dmac/MUX1
- U42 pad 4: /dmac0/A18/D10 -> /dmac/MUX2
- U42 pad 5: /dmac0/A19/D11 -> /dmac/MUX3
- U42 pad 6: /dmac0/A20/D12 -> /dmac/MUX4
- U42 pad 7: /dmac0/A21/D13 -> /dmac/MUX5
- U42 pad 8: /dmac0/A22/D14 -> /dmac/MUX6
- U42 pad 9: /dmac0/A23/D15 -> /dmac/MUX7
- U43 pad 1: /dmac0/~{OWN} -> /dmac/demuxer/~{OWN}
- U43 pad 11: /dmac0/UAS -> /dmac/demuxer/UAS
- U43 pad 12: A23 -> A15
- U43 pad 13: A22 -> A14
- U43 pad 14: A21 -> A13
- U43 pad 15: A20 -> A12
- U43 pad 16: A19 -> A11
- U43 pad 17: A18 -> A10
- U43 pad 18: A17 -> A9
- U43 pad 19: A16 -> A8
- U43 pad 2: /dmac0/A16/D8 -> /dmac/MUX0
- U43 pad 3: /dmac0/A17/D9 -> /dmac/MUX1
- U43 pad 4: /dmac0/A18/D10 -> /dmac/MUX2
- U43 pad 5: /dmac0/A19/D11 -> /dmac/MUX3
- U43 pad 6: /dmac0/A20/D12 -> /dmac/MUX4
- U43 pad 7: /dmac0/A21/D13 -> /dmac/MUX5
- U43 pad 8: /dmac0/A22/D14 -> /dmac/MUX6
- U43 pad 9: /dmac0/A23/D15 -> /dmac/MUX7
- U44 pad 1: +5V -> /dmac/demuxer/~{DDIR}
- U44 pad 10: +5V -> GND
- U44 pad 11: /dmac0/~{HALT0} -> D31
- U44 pad 12: /dmac0/~{BERR0} -> D30
- U44 pad 13: /dmac0/~{RETRY0} -> D29
- U44 pad 14: unconnected-(U44-GS-Pad14) -> D28
- U44 pad 15: unconnected-(U44-EO-Pad15) -> D27
- U44 pad 16: +5V -> D26
- U44 pad 2: +5V -> /dmac/MUX8
- U44 pad 3: +5V -> /dmac/MUX9
- U44 pad 4: ~{RST} -> /dmac/MUX10
- U44 pad 5: GND -> /dmac/MUX11
- U44 pad 6: /dmac0/~{BEC2} -> /dmac/MUX12
- U44 pad 7: /dmac0/~{BEC1} -> /dmac/MUX13
- U44 pad 8: GND -> /dmac/MUX14
- U44 pad 9: /dmac0/~{BEC0} -> /dmac/MUX15
- U5 pad 1: R/~{W} -> GND
- U5 pad 10: GND -> +5V
- U5 pad 11: D19 -> unconnected-(U5-NC-Pad11)
- U5 pad 12: D3 -> MA0
- U5 pad 13: D18 -> MA1
- U5 pad 14: D2 -> MA2
- U5 pad 15: D17 -> MA3
- U5 pad 16: D1 -> MA4
- U5 pad 17: D16 -> MA5
- U5 pad 18: D0 -> MA6
- U5 pad 19: GND -> MA10
- U5 pad 2: MD0 -> D0
- U5 pad 20: +5V -> D4
- U5 pad 3: MD16 -> D16
- U5 pad 4: MD1 -> D1
- U5 pad 5: MD17 -> D17
- U5 pad 6: MD2 -> D2
- U5 pad 7: MD18 -> D18
- U5 pad 8: MD3 -> D3
- U5 pad 9: MD19 -> D19
- U6 pad 2: MD0 -> D0
- U6 pad 20: MD4 -> D4
- U6 pad 21: MD20 -> D20
- U6 pad 22: MD5 -> D5
- U6 pad 23: MD21 -> D21
- U6 pad 24: MD6 -> D6
- U6 pad 25: MD22 -> D22
- U6 pad 26: MD7 -> D7
- U6 pad 27: MD23 -> D23
- U6 pad 3: MD16 -> D16
- U6 pad 33: /dram/~{RAS2} -> /dram/~{RAS0}
- U6 pad 34: /dram/~{RAS3} -> /dram/~{RAS1}
- U6 pad 4: MD1 -> D1
- U6 pad 44: /dram/~{RAS2} -> /dram/~{RAS0}
- U6 pad 45: /dram/~{RAS3} -> /dram/~{RAS1}
- U6 pad 49: MD8 -> D8
- U6 pad 5: MD17 -> D17
- U6 pad 50: MD24 -> D24
- U6 pad 51: MD9 -> D9
- U6 pad 52: MD25 -> D25
- U6 pad 53: MD10 -> D10
- U6 pad 54: MD26 -> D26
- U6 pad 55: MD11 -> D11
- U6 pad 56: MD27 -> D27
- U6 pad 57: MD12 -> D12
- U6 pad 58: MD28 -> D28
- U6 pad 6: MD2 -> D2
- U6 pad 60: MD29 -> D29
- U6 pad 61: MD13 -> D13
- U6 pad 62: MD30 -> D30
- U6 pad 63: MD14 -> D14
- U6 pad 64: MD31 -> D31
- U6 pad 65: MD15 -> D15
- U6 pad 7: MD18 -> D18
- U6 pad 8: MD3 -> D3
- U6 pad 9: MD19 -> D19
- U7 pad 1: GND -> A19
- U7 pad 10: +5V -> A3
- U7 pad 11: unconnected-(U7-NC-Pad11) -> A2
- U7 pad 12: MA0 -> A1
- U7 pad 13: MA1 -> D16
- U7 pad 14: MA2 -> D17
- U7 pad 15: MA3 -> D18
- U7 pad 16: MA4 -> GND
- U7 pad 17: MA5 -> D19
- U7 pad 18: MA6 -> D20
- U7 pad 19: MA10 -> D21
- U7 pad 2: MD0 -> A17
- U7 pad 20: MD4 -> D22
- U7 pad 21: MD20 -> D23
- U7 pad 22: MD5 -> ~{FLASH_CS}
- U7 pad 23: MD21 -> A11
- U7 pad 24: MD6 -> GND
- U7 pad 25: MD22 -> A12
- U7 pad 26: MD7 -> A10
- U7 pad 27: MD23 -> A9
- U7 pad 28: MA7 -> A14
- U7 pad 29: MA11 -> A15
- U7 pad 3: MD16 -> A16
- U7 pad 30: +5V -> A18
- U7 pad 31: MA8 -> unconnected-(U7-PGM-Pad31)
- U7 pad 32: MA9 -> +5V
- U7 pad 4: MD1 -> A13
- U7 pad 5: MD17 -> A8
- U7 pad 6: MD2 -> A7
- U7 pad 7: MD18 -> A6
- U7 pad 8: MD3 -> A5
- U7 pad 9: MD19 -> A4
- U8 pad 1: R/~{W} -> A19
- U8 pad 10: GND -> A3
- U8 pad 11: D24 -> A2
- U8 pad 12: D8 -> A1
- U8 pad 13: D25 -> D24
- U8 pad 14: D11 -> D25
- U8 pad 16: D9 -> GND
- U8 pad 18: D10 -> D28
- U8 pad 19: GND -> D29
- U8 pad 2: MD8 -> A17
- U8 pad 20: +5V -> D30
- U8 pad 3: MD24 -> A16
- U8 pad 4: MD9 -> A13
- U8 pad 5: MD25 -> A8
- U8 pad 6: MD10 -> A7
- U8 pad 7: MD26 -> A6
- U8 pad 8: MD11 -> A5
- U8 pad 9: MD27 -> A4
- U9 pad 1: R/~{W} -> Net-(U9-C1+)
- U9 pad 10: GND -> /serial/~{RTSA}
- U9 pad 11: D20 -> /serial/TxDA
- U9 pad 12: D4 -> /serial/RxDA
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Routing:
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- removed copper zone on In2.Cu, net GNDA
Other:
- board outline added: 254 x 254 mm
